File: designs/ad7606-two-channel-icm42688/hardware/main/afo_revb_main.kicad_sch (KiCad schematic)
At the start: 106 parts, among them J1 USB-C (battery powered), J10 Expansion, J2 microSD, J3 FOOT IMU, J4 SHANK IMU, J5 EMG1, J6 EMG2, J9 PROTECTED 1S BATTERY, Q1 DMP2035U, Q2 2N7002, SW1 POWER, SW2 BOOT, SW3 EN, SW4 BUTTON, U1 ESP32-S3-WROOM-1-N8R8, U2 AD7606BSTZ, U3 MCP6004T-I/ST, U4 MCP6004T-I/ST, U5 MCP6001T-I/OT, U6 TPS63070RNMR, U7 TPS7A2030PDBVR, U8 TPS60150DRVR

Commit message: Hold the AD7606 in shutdown until both rails are up (PCB + firmware 1.11)
AVCC is generated from 3V3D by the TPS60150, so VDRIVE always leads AVCC at
power-up, against the absolute-maximum rating and ADI AN-1091. As approved
by the project lead:

- PCB: AD7606 STBY (pin 7) moves from 3V3D to ADC_STBY on ESP32 GPIO14 with
  a 100 k pull-down (R70), keeping the converter in full shutdown with RANGE
  low; a BAT760 Schottky (D30) from 3V3D to 5V_ADC limits VDRIVE - AVCC while
  the charge pump starts. New copper routed against the existing board; the
  RANGE (pin 8) ground tie that blocked pin 7 now has its own ground via.
  DRC 0 violations / 0 unconnected, ERC 0, connection audit and package
  validator pass; manufacturing exports regenerated. Not yet built.
- Firmware ad7606-2ch-1.11: PCB builds release STBY once per boot, wait the
  30 ms shutdown wake-up, then reset the ADC; breadboard builds unchanged.
  Nine profiles rebuilt; driver test covers the ordering.
- Wokwi web editor on the 1.11 integrated image: nominal, write-delay and
  USB-attached cases pass with the production converter and live decoder;
  the remaining 15 cases are pending. Fixture PSRAM budget and UDP buffer
  updated for the 1.7+ queue and 1,400-byte metadata limit.
- Lab kit repackaged (160a349a) and verified.

Co-Authored-By: Claude Opus 5.5 <noreply@anthropic.com>
Parts:
- added D30: BAT760, Diode_SMD:D_SOD-323, symbol RevB:D30
- added R70: 100k, Resistor_SMD:R_0603_1608Metric, symbol RevB:R70
Connections:
- net 3V3D: now also D30.2 (A); no longer U2.7 (STBY_N)
- net 5V_ADC: now also D30.1 (K)
- net GND: now also R70.2 (GND)
- net ADC_STBY: now reaches U1.22 (GPIO14)
- net ADC_STBY: now also U2.7 (STBY_N), R70.1 (ADC_STBY)
- no-connect marks 16 -> 15
