File: designs/ad7606-two-channel-mpu6050/hardware/main/afo_revb_main.kicad_pcb (KiCad board)
At the start: 4 copper layers, 75 x 50 mm, 106 parts, among them J1 USB-C (battery powered), J10 Expansion, J2 microSD, J3 FOOT MPU6050, J4 SHANK MPU6050, J5 EMG1, J6 EMG2, J9 PROTECTED 1S BATTERY, Q1 DMP2035U, Q2 2N7002, SW1 POWER, SW2 BOOT, SW3 EN, SW4 BUTTON, U1 ESP32-S3-WROOM-1-N8R8, U2 AD7606BSTZ, U3 MCP6004T-I/ST, U4 MCP6004T-I/ST, U5 MCP6001T-I/OT, U6 TPS63070RNMR, U7 TPS7A2030PDBVR, U8 TPS60150DRVR

Commit message: Port the AD7606 supply-ramp fix to the other AD7606 designs
The expandable ICM, expandable MPU-6050 and two-channel MPU-6050 boards share
the fixed-two power topology (TPS60150 AVCC from 3V3D, STBY tied to 3V3D,
GPIO14 free). Apply the same change: STBY on GPIO14 with a 100 k pull-down
(R70), BAT760 (D30) from 3V3D to 5V_ADC, and the RANGE ground tie re-routed
so pin 7 can escape. DRC 0 violations / 0 unconnected and ERC 0 on each
board; package validators pass; manufacturing and viewer files re-exported.

Firmware dual-1.4 / mpu6050-1.4: PCB builds release STBY, wait 30 ms and
reset (ADI AN-1091); the ADC driver matches the tested fixed-two driver and
its native test passes against each design's board.h. 27 profiles rebuilt;
host tests pass. ADS131M04 designs unchanged (TI allows any supply order).
Parts:
- added D30: BAT760, Diode_SMD:D_SOD-323, F.Cu at (38.9, 19.6)
- added R70: 100k, Resistor_SMD:R_0603_1608Metric, F.Cu at (23.6, 27.4)
Connections:
- U1 pad 22: (no net) -> ADC_STBY
- U2 pad 7: 3V3D -> ADC_STBY
Routing:
- net ADC_STBY: track 0.00 -> 48.9 mm, vias 0 -> 7
- net 3V3D: track 268.3 -> 271.8 mm, vias 13 -> 14
- net 5V_ADC: track 61.5 -> 62.2 mm
- net GND: track 449.1 -> 449.5 mm, vias 14 -> 16
